File: circuit/circuit.kicad_sch (KiCad schematic)
At the start: 0 parts

Commit message: Finish basic schematic
Other:
- added sheet Audio (audio.kicad_sch)
- added sheet WIFI & BT (wifi&bt.kicad_sch)
- added sheet controller (controller.kicad_sch)
- added sheet power (power.kicad_sch)
Changed lines of the file:
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@@
-(kicad_sch (version 20211123) (generator eeschema)
+(kicad_sch (version 20230121) (generator eeschema)
   (paper "A4")
   (title_block
     (title "Allwinner V3s")
-    (date "2022-09-02")
+    (date "2023-08-02")
     (rev "1.0.1")
   )
+  (sheet (at 77.47 115.57) (size 25.4 33.02) (fields_autoplaced)
+    (stroke (width 0.1524) (type solid))
+    (fill (color 0 0 0 0.0000))
+    (property "Sheetname" "WIFI & BT" (at 77.47 114.8584 0)
+      (effects (font (size 1.27 1.27)) (justify left bottom))
+    )
+    (property "Sheetfile" "wifi&bt.kicad_sch" (at 77.47 149.1746 0)
+      (effects (font (size 1.27 1.27)) (justify left top))
+    )
+    (instances
+      (project "circuit"
+        (path "/d348603e-ed7b-41d8-b24d-7293f9d8c9fb" (page "4"))
+      )
+    )
+  )
+  (sheet (at 113.03 38.1) (size 85.09 8.89) (fields_autoplaced)
+    (stroke (width 0.1524) (type solid))
+    (fill (color 0 0 0 0.0000))
+    (property "Sheetname" "power" (at 113.03 37.3884 0)
+      (effects (font (size 1.27 1.27)) (justify left bottom))
+    )
+    (property "Sheetfile" "power.kicad_sch" (at 113.03 47.5746 0)
+      (effects (font (size 1.27 1.27)) (justify left top) hide)
+    )
+    (instances
+      (project "circuit"
+        (path "/d348603e-ed7b-41d8-b24d-7293f9d8c9fb" (page "3"))
+      )
+    )
+  )
+  (sheet (at 113.03 55.88) (size 85.09 92.71) (fields_autoplaced)
+    (stroke (width 0.1524) (type solid))
+    (fill (color 0 0 0 0.0000))
+    (property "Sheetname" "controller" (at 113.03 55.1684 0)
+      (effects (font (size 1.27 1.27)) (justify left bottom))
+    )
+    (property "Sheetfile" "controller.kicad_sch" (at 113.03 149.1746 0)
+      (effects (font (size 1.27 1.27)) (justify left top) hide)
+    )
+    (pin "LCD_HSYNC" output (at 113.03 64.77 180)
+      (effects (font (size 1.27 1.27)) (justify left))
+    )
+    (pin "LCD_D2" output (at 113.03 72.39 180)
+      (effects (font (size 1.27 1.27)) (justify left))
+    )
+    (pin "LCD_VSYNC" output (at 113.03 67.31 180)
+      (effects (font (size 1.27 1.27)) (justify left))
+    )
+    (pin "LCD_DE" output (at 113.03 62.23 180)
+      (effects (font (size 1.27 1.27)) (justify left))
+    )
+    (pin "LCD_CLK" output (at 113.03 59.69 180)
+      (effects (font (size 1.27 1.27)) (justify left))
+    )
+    (pin "LCD_D11" output (at 113.03 90.17 180)
+      (effects (font (size 1.27 1.27)) (justify left))
+    )
+    (pin "LCD_D10" output (at 113.03 87.63 180)
+      (effects (font (size 1.27 1.27)) (justify left))
+    )
+    (pin "LCD_D12" output (at 113.03 92.71 180)
+      (effects (font (size 1.27 1.27)) (justify left))
+    )
+    (pin "LCD_D7" output (at 113.03 85.09 180)
+      (effects (font (size 1.27 1.27)) (justify left))
+    )
+    (pin "LCD_D6" output (at 113.03 82.55 180)
+      (effects (font (size 1.27 1.27)) (justify left))
+    )
+    (pin "LCD_D4" output (at 113.03 77.47 180)
+      (effects (font (size 1.27 1.27)) (justify left))
+    )
+    (pin "LCD_D5" output (at 113.03 80.01 180)
+      (effects (font (size 1.27 1.27)) (justify left))
+    )
+    (pin "LCD_D3" output (at 113.03 74.93 180)
+      (effects (font (size 1.27 1.27)) (justify left))
+    )
+    (pin "LCD_D23" output (at 113.03 115.57 180)
+      (effects (font (size 1.27 1.27)) (justify left))
+    )
+    (pin "LCD_D22" output (at 113.03 113.03 180)
+      (effects (font (size 1.27 1.27)) (justify left))
+    )
+    (pin "LCD_D21" output (at 113.03 110.49 180)
+      (effects (font (size 1.27 1.27)) (justify left))
+    )
+    (pin "LCD_D20" output (at 113.03 107.95 180)
+      (effects (font (size 1.27 1.27)) (justify left))
+    )
+    (pin "LCD_D19" output (at 113.03 105.41 180)
+      (effects (font (size 1.27 1.27)) (justify left))
+    )
+    (pin "LCD_D14" output (at 113.03 97.79 180)
+      (effects (font (size 1.27 1.27)) (justify left))
+    )
+    (pin "LCD_D18" output (at 113.03 102.87 180)
+      (effects (font (size 1.27 1.27)) (justify left))
+    )
+    (pin "LCD_D15" output (at 113.03 100.33 180)
+      (effects (font (size 1.27 1.27)) (justify left))
+    )
+    (pin "LCD_D13" output (at 113.03 95.25 180)
+      (effects (font (size 1.27 1.27)) (justify left))
+    )
+    (pin "EPHY_LEDL" output (at 198.12 59.69 0)
+      (effects (font (size 1.27 1.27)) (justify right))
+    )
+    (pin "EPHY_LEDS" output (at 198.12 62.23 0)
+      (effects (font (size 1.27 1.27)) (justify right))
+    )
+    (pin "EPHY_TXN" output (at 198.12 64.77 0)
+      (effects (font (size 1.27 1.27)) (justify right))
+    )
+    (pin "EPHY_TXP" output (at 198.12 67.31 0)
+      (effects (font (size 1.27 1.27)) (justify right))
+    )
+    (pin "EPHY_RXP" input (at 198.12 69.85 0)
+      (effects (font (size 1.27 1.27)) (justify right))
+    )
+    (pin "EPHY_RXN" input (at 198.12 72.39 0)
+      (effects (font (size 1.27 1.27)) (justify right))
+    )
+    (pin "KEYADC" output (at 198.12 138.43 0)
+      (effects (font (size 1.27 1.27)) (justify right))
+    )
+    (pin "USBDM" output (at 198.12 115.57 0)
+      (effects (font (size 1.27 1.27)) (justify right))
+    )
+    (pin "USBDP" bidirectional (at 198.12 118.11 0)
+      (effects (font (size 1.27 1.27)) (justify right))
+    )
+    (pin "SDC1_D2" bidirectional (at 113.03 130.81 180)
+      (effects (font (size 1.27 1.27)) (justify left))
+    )
+    (pin "SDC1_D1" bidirectional (at 113.03 128.27 180)
+      (effects (font (size 1.27 1.27)) (justify left))
+    )
+    (pin "SDC1_D0" bidirectional (at 113.03 125.73 180)
+      (effects (font (size 1.27 1.27)) (justify left))
+    )
+    (pin "SDC1_CMD" output (at 113.03 123.19 180)
+      (effects (font (size 1.27 1.27)) (justify left))
+    )
+    (pin "SDC1_CLK" output (at 113.03 120.65 180)
+      (effects (font (size 1.27 1.27)) (justify left))
+    )
+    (pin "SPI_CLK" output (at 198.12 105.41 0)
+      (effects (font (size 1.27 1.27)) (justify right))
+    )
+    (pin "SPI_CS" output (at 198.12 102.87 0)
+      (effects (font (size 1.27 1.27)) (justify right))
+    )
+    (pin "SPI_MOSI" output (at 198.12 107.95 0)
+      (effects (font (size 1.27 1.27)) (justify right))
+    )
+    (pin "UART0_RX" input (at 198.12 90.17 0)
+      (effects (font (size 1.27 1.27)) (justify right))
+    )
+    (pin "UART0_TX" output (at 198.12 92.71 0)
+      (effects (font (size 1.27 1.27)) (justify right))
+    )
+    (pin "SPI_MISO" input (at 198.12 110.49 0)
+      (effects (font (size 1.27 1.27)) (justify right))
+    )
+    (pin "SDC1_D3" bidirectional (at 113.03 133.35 180)
+      (effects (font (size 1.27 1.27)) (justify left))
+    )
+    (pin "TWI0_CLK" output (at 198.12 123.19 0)
+      (effects (font (size 1.27 1.27)) (justify right))
+    )
+    (pin "TWI0_SDA" bidirectional (at 198.12 125.73 0)
+      (effects (font (size 1.27 1.27)) (justify right))
+    )
+    (pin "UART1_TX" output (at 198.12 97.79 0)
+      (effects (font (size 1.27 1.27)) (justify right))
+    )
+    (pin "UART1_RX" input (at 198.12 95.25 0)
+      (effects (font (size 1.27 1.27)) (justify right))
+    )
+    (pin "PWM0" output (at 198.12 130.81 0)
+      (effects (font (size 1.27 1.27)) (justify right))
+    )
+    (pin "PWM1" output (at 198.12 133.35 0)
+      (effects (font (size 1.27 1.27)) (justify right))
+    )
+    (pin "UART2_RX" input (at 113.03 143.51 180)
+      (effects (font (size 1.27 1.27)) (justify left))
+    )
+    (pin "UART2_TX" output (at 113.03 146.05 180)
+      (effects (font (size 1.27 1.27)) (justify left))
+    )
+    (pin "MIC_N" bidirectional (at 198.12 77.47 0)
+      (effects (font (size 1.27 1.27)) (justify right))
+    )
+    (pin "MIC_P" bidirectional (at 198.12 80.01 0)
+      (effects (font (size 1.27 1.27)) (justify right))
+    )
+    (pin "HP_L" bidirectional (at 198.12 82.55 0)
+      (effects (font (size 1.27 1.27)) (justify right))
+    )
+    (pin "HP_R" bidirectional (at 198.12 85.09 0)
+      (effects (font (size 1.27 1.27)) (justify right))
+    )
+    (pin "UART2_RTS" bidirectional (at 113.03 138.43 180)
+      (effects (font (size 1.27 1.27)) (justify left))
+    )
+    (pin "UART2_CTS" bidirectional (at 113.03 140.97 180)
+      (effects (font (size 1.27 1.27)) (justify left))
+    )
+    (instances
+      (project "circuit"
+        (path "/d348603e-ed7b-41d8-b24d-7293f9d8c9fb" (page "2"))
+      )
+    )
+  )
+  (sheet (at 204.47 72.39) (size 25.4 19.05) (fields_autoplaced)
+    (stroke (width 0.1524) (type solid))
+    (fill (color 0 0 0 0.0000))
+    (property "Sheetname" "Audio" (at 204.47 71.6784 0)
+      (effects (font (size 1.27 1.27)) (justify left bottom))
+    )
+    (property "Sheetfile" "audio.kicad_sch" (at 204.47 92.0246 0)
+      (effects (font (size 1.27 1.27)) (justify left top))
+    )
+    (instances
+      (project "circuit"
+        (path "/d348603e-ed7b-41d8-b24d-7293f9d8c9fb" (page "5"))
+      )
+    )
+  )
   (sheet_instances
